File: kicad/stepper_driver/driver.sch (KiCad schematic (older format))
At the start: 45 parts, among them U14 MCP23S18, U15 TB6560AHQ, U16 TB6560AHQ

Commit message: stepper_driver: new revision
Forgot the history on this one. If anybody is watching. Sorry :(
Moved datahseets into project folder.
I guess I've added some footprints too.

Signed-off-by: Gratian Crisan <gratian.crisan@ni.com>
Parts:
- removed C10, C9: 0.1uF, symbol C
- removed R16, R17: 3k, Resistors_SMD:R_1206, symbol R
- C10: renamed from C12; footprint (none) -> Capacitors_SMD:C_0805_HandSoldering
- C11: renamed from C13; footprint (none) -> Capacitors_SMD:C_1206_HandSoldering
- C12: renamed from C14; footprint (none) -> Capacitors_SMD:C_1206_HandSoldering
- C13: renamed from C15; footprint (none) -> Capacitors_SMD:c_elec_4x5.3
- C14: renamed from C16; footprint (none) -> Capacitors_SMD:c_elec_4x5.3
- C15: renamed from C17; footprint (none) -> Capacitors_SMD:C_1206_HandSoldering
- C16: renamed from C18; footprint (none) -> Capacitors_SMD:C_1206_HandSoldering
- C17: renamed from C19; footprint (none) -> Capacitors_SMD:c_elec_4x5.3
- C18: renamed from C20; footprint (none) -> Capacitors_SMD:c_elec_4x5.3
- C8: footprint (none) -> Capacitors_SMD:C_1206_HandSoldering
- C9: renamed from C11; footprint (none) -> Capacitors_SMD:C_0805_HandSoldering
- D1, D2: footprint (none) -> LEDs:LED-3MM
- D10, D11, D12, D13, D14, D15, D16, D17, D18, D3, D4, D5, D6, D7, D8, D9: footprint (none) -> footprints:SMD-Mini2-F3-B
- F1, F2: footprint (none) -> footprints:Fuse_SMD2410
- R15: footprint (none) -> Resistors_SMD:R_1206_HandSoldering
- R16: renamed from R18; footprint (none) -> Resistors_SMD:R_1206_HandSoldering
- R17: renamed from R19; footprint (none) -> Resistors_SMD:R_1206_HandSoldering
- R18: renamed from R20; footprint (none) -> Resistors_SMD:R_1206_HandSoldering
- R19: renamed from R21; footprint (none) -> Resistors_SMD:R_1206_HandSoldering
- R20: renamed from R22; footprint (none) -> Resistors_SMD:R_1206_HandSoldering
- R21: renamed from R23; footprint (none) -> Resistors_SMD:R_1206_HandSoldering
- U14: footprint (none) -> SMD_Packages:SOIC-28
- U15, U16: footprint (none) -> footprints:HZIP25-P-1.27
Connections:
- net +12V: now also D11.1 (K), D13.1 (K), D15.1 (K), D17.1 (K), D3.1 (K), D5.1 (K), D7.1 (K), D9.1 (K); no longer D11.2 (A), D13.2 (A), D15.2 (A), D17.2 (A), D3.2 (A), D5.2 (A), D7.2 (A), D9.2 (A)
- net AM0: now also D7.2 (A), D8.1 (K); no longer D7.1 (K), D8.2 (A)
- net AM1: now also D10.1 (K), D9.2 (A); no longer D10.2 (A), D9.1 (K)
- net AP0: now also D3.2 (A), D4.1 (K); no longer D3.1 (K), D4.2 (A)
- net AP1: now also D5.2 (A), D6.1 (K); no longer D5.1 (K), D6.2 (A)
- net BM0: now also D11.2 (A), D12.1 (K); no longer D11.1 (K), D12.2 (A)
- net BM1: now also D13.2 (A), D14.1 (K); no longer D13.1 (K), D14.2 (A)
- net BP0: now also D15.2 (A), D16.1 (K); no longer D15.1 (K), D16.2 (A)
- net BP1: now also D17.2 (A), D18.1 (K); no longer D17.1 (K), D18.2 (A)
- net CH0_ENA: now also U14.20 (GPA0); no longer U14.22 (GPA2)
- net CH0_TQ2: now also U14.21 (GPA1); no longer U14.20 (GPA0)
- net CH1_ENA: now also U14.3 (GPB0); no longer U14.5 (GPB2)
- net CH1_TQ2: now also U14.4 (GPB1); no longer U14.3 (GPB0)
- net GND: now also D10.2 (A), D12.2 (A), D14.2 (A), D16.2 (A), D18.2 (A), D4.2 (A), D6.2 (A), D8.2 (A); no longer D10.1 (K), D12.1 (K), D14.1 (K), D16.1 (K), D18.1 (K), D4.1 (K), D6.1 (K), D8.1 (K)
- net at U14.10 (GPB7): now also U16.22 (M2); no longer U16.3 (CLK)
- net at U14.23 (GPA3): now also U15.5 (~RESET); no longer U15.22 (M2)
- net at U14.24 (GPA4): now also U15.17 (MO); no longer U15.23 (M1)
- net at U14.26 (GPA6): now also U15.23 (M1); no longer U15.17 (MO)
- net at U15.3 (CLK): now also U14.22 (GPA2); no longer U14.27 (GPA7)
- net at U14.6 (GPB3): now also U16.5 (~RESET); no longer U16.22 (M2)
- net at U14.7 (GPB4): now also U16.17 (MO); no longer U16.23 (M1)
- net at U14.9 (GPB6): now also U16.23 (M1); no longer U16.17 (MO)
- net CH0_TQ1: no longer names the net of U15.2 (TQ1)
- net CH0_TQ1: no longer U14.21 (GPA1)
- net CH1_TQ1: no longer names the net of U16.2 (TQ1)
- net CH1_TQ1: no longer U14.4 (GPB1)
- net NC: no longer names the net of U14.18 (INTB)
- new net: U14.27 (GPA7), U15.22 (M2)
- new net: U14.5 (GPB2), U16.3 (CLK)
- no-connect marks 0 -> 7
Other:
- moved on the sheet: U14
