File: kicad/stepper_driver/in_isolation.sch (KiCad schematic (older format))
At the start: 5 parts, among them U2 SN74LVC1G14DBV, U3 6N137S

Commit message: stepper_driver: new revision
Forgot the history on this one. If anybody is watching. Sorry :(
Moved datahseets into project folder.
I guess I've added some footprints too.

Signed-off-by: Gratian Crisan <gratian.crisan@ni.com>
Parts:
- C2: footprint (none) -> Capacitors_SMD:C_1206_HandSoldering
- R3, R4: footprint (none) -> Resistors_SMD:R_1206_HandSoldering
- U2: footprint (none) -> footprints:SOT-23-5
- U3: footprint (none) -> footprints:SMD-8
Changed lines of the file:
@@
 EESchema Schematic File Version 2
+LIBS:stepper_driver-rescue
 LIBS:power
 LIBS:device
@@
 LIBS:custom
 LIBS:stepper_driver-cache
-EELAYER 25 0
+EELAYER 26 0
 EELAYER END
 $Descr A4 11693 8268
 encoding utf-8
 Sheet 2 10
-Title "CMOS INPUT TTL OUTPUT OPTO ISOLATION"
-Date "Sun 22 Mar 2015"
+Title "Quad Stepper Motor Driver"
+Date "2016-12-15"
 Rev "1.0"
-Comp ""
+Comp "Gratian & co."
 Comment1 ""
 Comment2 ""
@@
 AR Path="/55139FA9/5510850A" Ref="U11"  Part="1"
 AR Path="/5510BF5A/5510850A" Ref="U21"  Part="1"
-F 0 "U3" H 6200 3750 60  0000 C CNN
+F 0 "U21" H 6200 3750 60  0000 C CNN
 F 1 "6N137S" H 6200 4250 60  0000 C CNN
-F 2 "" H 6200 4000 60  0000 C CNN
+F 2 "footprints:SMD-8" H 6200 4000 60  0001 C CNN
 F 3 "" H 6200 4000 60  0000 C CNN
 	1    6200 4000
@@
 $EndComp
 $Comp
-L +3.3V #PWR036
+L +3.3V #PWR039
 U 1 1 55108511
 P 5400 3700
-AR Path="/55107C90/55108511" Ref="#PWR036"  Part="1"
-AR Path="/5510B4E2/55108511" Ref="#PWR043"  Part="1"
-AR Path="/5512F1A5/55108511" Ref="#PWR058"  Part="1"
-AR Path="/55139FA9/55108511" Ref="#PWR065"  Part="1"
-AR Path="/5510BF5A/55108511" Ref="#PWR0144"  Part="1"
-F 0 "#PWR0144" H 5400 3550 50  0001 C CNN
+AR Path="/55107C90/55108511" Ref="#PWR039"  Part="1"
+AR Path="/5510B4E2/55108511" Ref="#PWR046"  Part="1"
+AR Path="/5512F1A5/55108511" Ref="#PWR061"  Part="1"
+AR Path="/55139FA9/55108511" Ref="#PWR068"  Part="1"
+AR Path="/5510BF5A/55108511" Ref="#PWR0113"  Part="1"
+F 0 "#PWR0113" H 5400 3550 50  0001 C CNN
 F 1 "+3.3V" H 5400 3840 50  0000 C CNN
 F 2 "" H 5400 3700 60  0000 C CNN
@@
 AR Path="/55139FA9/55108517" Ref="U10"  Part="1"
 AR Path="/5510BF5A/55108517" Ref="U20"  Part="1"
-F 0 "U2" H 4850 3550 60  0000 C CNN
+F 0 "U20" H 4850 3550 60  0000 C CNN
 F 1 "SN74LVC1G14DBV" H 4850 4150 60  0000 C CNN
-F 2 "" H 4700 4150 60  0000 C CNN
+F 2 "footprints:SOT-23-5" H 4700 4150 60  0001 C CNN
 F 3 "" H 4700 4150 60  0000 C CNN
 	1    4850 3850
@@
 AR Path="/5512F1A5/55108520" Ref="R9"  Part="1"
 AR Path="/55139FA9/55108520" Ref="R11"  Part="1"
-AR Path="/5510BF5A/55108520" Ref="R33"  Part="1"
-F 0 "R3" V 5580 3950 50  0000 C CNN
+AR Path="/5510BF5A/55108520" Ref="R29"  Part="1"
+F 0 "R29" V 5580 3950 50  0000 C CNN
 F 1 "220" V 5500 3950 50  0000 C CNN
-F 2 "" V 5430 3950 30  0000 C CNN
+F 2 "Resistors_SMD:R_1206_HandSoldering" V 5430 3950 30  0001 C CNN
 F 3 "" H 5500 3950 30  0000 C CNN
 	1    5500 3950
@@
 	5750 3950 5650 3950
 $Comp
-L GND #PWR037
+L GND #PWR040
 U 1 1 55108529
 P 4350 4200
-AR Path="/55107C90/55108529" Ref="#PWR037"  Part="1"
-AR Path="/5510B4E2/55108529" Ref="#PWR044"  Part="1"
-AR Path="/5512F1A5/55108529" Ref="#PWR059"  Part="1"
-AR Path="/55139FA9/55108529" Ref="#PWR066"  Part="1"
-AR Path="/5510BF5A/55108529" Ref="#PWR0145"  Part="1"
-F 0 "#PWR0145" H 4350 3950 50  0001 C CNN
+AR Path="/55107C90/55108529" Ref="#PWR040"  Part="1"
+AR Path="/5510B4E2/55108529" Ref="#PWR047"  Part="1"
+AR Path="/5512F1A5/55108529" Ref="#PWR062"  Part="1"
+AR Path="/55139FA9/55108529" Ref="#PWR069"  Part="1"
+AR Path="/5510BF5A/55108529" Ref="#PWR0114"  Part="1"
+F 0 "#PWR0114" H 4350 3950 50  0001 C CNN
 F 1 "GND" H 4350 4050 50  0000 C CNN
 F 2 "" H 4350 4200 60  0000 C CNN
@@
 	4450 4000 4350 4000
 $Comp
-L GND #PWR038
+L GND #PWR041
 U 1 1 55108530
 P 5600 4250
-AR Path="/55107C90/55108530" Ref="#PWR038"  Part="1"
-AR Path="/5510B4E2/55108530" Ref="#PWR045"  Part="1"
-AR Path="/5512F1A5/55108530" Ref="#PWR060"  Part="1"
-AR Path="/55139FA9/55108530" Ref="#PWR067"  Part="1"
-AR Path="/5510BF5A/55108530" Ref="#PWR0146"  Part="1"
-F 0 "#PWR0146" H 5600 4000 50  0001 C CNN
+AR Path="/55107C90/55108530" Ref="#PWR041"  Part="1"
+AR Path="/5510B4E2/55108530" Ref="#PWR048"  Part="1"
+AR Path="/5512F1A5/55108530" Ref="#PWR063"  Part="1"
+AR Path="/55139FA9/55108530" Ref="#PWR070"  Part="1"
+AR Path="/5510BF5A/55108530" Ref="#PWR0115"  Part="1"
+F 0 "#PWR0115" H 5600 4000 50  0001 C CNN
 F 1 "GND" H 5600 4100 50  0000 C CNN
 F 2 "" H 5600 4250 60  0000 C CNN
@@
 $EndComp
 $Comp
-L +5V #PWR039
+L +5V #PWR042
 U 1 1 55108537
 P 6750 3700
-AR Path="/55107C90/55108537" Ref="#PWR039"  Part="1"
-AR Path="/5510B4E2/55108537" Ref="#PWR046"  Part="1"
-AR Path="/5512F1A5/55108537" Ref="#PWR061"  Part="1"
-AR Path="/55139FA9/55108537" Ref="#PWR068"  Part="1"
-AR Path="/5510BF5A/55108537" Ref="#PWR0147"  Part="1"
-F 0 "#PWR0147" H 6750 3550 50  0001 C CNN
+AR Path="/55107C90/55108537" Ref="#PWR042"  Part="1"
+AR Path="/5510B4E2/55108537" Ref="#PWR049"  Part="1"
+AR Path="/5512F1A5/55108537" Ref="#PWR064"  Part="1"
+AR Path="/55139FA9/55108537" Ref="#PWR071"  Part="1"
+AR Path="/5510BF5A/55108537" Ref="#PWR0116"  Part="1"
+F 0 "#PWR0116" H 6750 3550 50  0001 C CNN
 F 1 "+5V" H 6750 3840 50  0000 C CNN
 F 2 "" H 6750 3700 60  0000 C CNN
@@
 Connection ~ 6750 3850
 $Comp
-L GND #PWR040
+L GND #PWR043
 U 1 1 55108543
 P 6750 4250
-AR Path="/55107C90/55108543" Ref="#PWR040"  Part="1"
-AR Path="/5510B4E2/55108543" Ref="#PWR047"  Part="1"
-AR Path="/5512F1A5/55108543" Ref="#PWR062"  Part="1"
-AR Path="/55139FA9/55108543" Ref="#PWR069"  Part="1"
-AR Path="/5510BF5A/55108543" Ref="#PWR0148"  Part="1"
-F 0 "#PWR0148" H 6750 4000 50  0001 C CNN
+AR Path="/55107C90/55108543" Ref="#PWR043"  Part="1"
+AR Path="/5510B4E2/55108543" Ref="#PWR050"  Part="1"
+AR Path="/5512F1A5/55108543" Ref="#PWR065"  Part="1"
+AR Path="/55139FA9/55108543" Ref="#PWR072"  Part="1"
+AR Path="/5510BF5A/55108543" Ref="#PWR0117"  Part="1"
+F 0 "#PWR0117" H 6750 4000 50  0001 C CNN
 F 1 "GND" H 6750 4100 50  0000 C CNN
 F 2 "" H 6750 4250 60  0000 C CNN
@@
 AR Path="/5512F1A5/5510854B" Ref="R10"  Part="1"
 AR Path="/55139FA9/5510854B" Ref="R12"  Part="1"
-AR Path="/5510BF5A/5510854B" Ref="R34"  Part="1"
-F 0 "R4" V 6980 3900 50  0000 C CNN
+AR Path="/5510BF5A/5510854B" Ref="R30"  Part="1"
+F 0 "R30" V 6980 3900 50  0000 C CNN
 F 1 "220" V 6900 3900 50  0000 C CNN
-F 2 "" V 6830 3900 30  0000 C CNN
+F 2 "Resistors_SMD:R_1206_HandSoldering" V 6830 3900 30  0001 C CNN
 F 3 "" H 6900 3900 30  0000 C CNN
 	1    6900 3900
@@
 AR Path="/5512F1A5/55108559" Ref="C5"  Part="1"
 AR Path="/55139FA9/55108559" Ref="C6"  Part="1"
-AR Path="/5510BF5A/55108559" Ref="C34"  Part="1"
-F 0 "C2" H 7825 4100 50  0000 L CNN
+AR Path="/5510BF5A/55108559" Ref="C30"  Part="1"
+F 0 "C30" H 7825 4100 50  0000 L CNN
 F 1 "0.1uF" H 7825 3900 50  0000 L CNN
-F 2 "" H 7838 3850 30  0000 C CNN
+F 2 "Capacitors_SMD:C_1206_HandSoldering" H 7838 3850 30  0001 C CNN
 F 3 "" H 7800 4000 60  0000 C CNN
 	1    7800 4000
@@
 OUT_TTL
 $Comp
-L GND #PWR041
+L GND #PWR044
 U 1 1 55108CC5
 P 7800 4250
-AR Path="/55107C90/55108CC5" Ref="#PWR041"  Part="1"
-AR Path="/5510B4E2/55108CC5" Ref="#PWR048"  Part="1"
-AR Path="/5512F1A5/55108CC5" Ref="#PWR063"  Part="1"
-AR Path="/55139FA9/55108CC5" Ref="#PWR070"  Part="1"
-AR Path="/5510BF5A/55108CC5" Ref="#PWR0149"  Part="1"
-F 0 "#PWR0149" H 7800 4000 50  0001 C CNN
+AR Path="/55107C90/55108CC5" Ref="#PWR044"  Part="1"
+AR Path="/5510B4E2/55108CC5" Ref="#PWR051"  Part="1"
+AR Path="/5512F1A5/55108CC5" Ref="#PWR066"  Part="1"
+AR Path="/55139FA9/55108CC5" Ref="#PWR073"  Part="1"
+AR Path="/5510BF5A/55108CC5" Ref="#PWR0118"  Part="1"
+F 0 "#PWR0118" H 7800 4000 50  0001 C CNN
 F 1 "GND" H 7800 4100 50  0000 C CNN
 F 2 "" H 7800 4250 60  0000 C CNN
@@
 $EndComp
 $Comp
-L +5V #PWR042
+L +5V #PWR045
 U 1 1 55108CDA
 P 7800 3700
-AR Path="/55107C90/55108CDA" Ref="#PWR042"  Part="1"
-AR Path="/5510B4E2/55108CDA" Ref="#PWR049"  Part="1"
-AR Path="/5512F1A5/55108CDA" Ref="#PWR064"  Part="1"
-AR Path="/55139FA9/55108CDA" Ref="#PWR071"  Part="1"
-AR Path="/5510BF5A/55108CDA" Ref="#PWR0150"  Part="1"
-F 0 "#PWR0150" H 7800 3550 50  0001 C CNN
+AR Path="/55107C90/55108CDA" Ref="#PWR045"  Part="1"
+AR Path="/5510B4E2/55108CDA" Ref="#PWR052"  Part="1"
+AR Path="/5512F1A5/55108CDA" Ref="#PWR067"  Part="1"
+AR Path="/55139FA9/55108CDA" Ref="#PWR074"  Part="1"
+AR Path="/5510BF5A/55108CDA" Ref="#PWR0119"  Part="1"
+F 0 "#PWR0119" H 7800 3550 50  0001 C CNN
 F 1 "+5V" H 7800 3840 50  0000 C CNN
 F 2 "" H 7800 3700 60  0000 C CNN
