File: kicad/stepper_driver/out_isolation.sch (KiCad schematic (older format))
At the start: 5 parts, among them U6 6N137S, U7 SN74LVC1G240DBVR

Commit message: stepper_driver: new revision
Forgot the history on this one. If anybody is watching. Sorry :(
Moved datahseets into project folder.
I guess I've added some footprints too.

Signed-off-by: Gratian Crisan <gratian.crisan@ni.com>
Parts:
- C4: footprint (none) -> Capacitors_SMD:C_1206_HandSoldering
- R7, R8: footprint (none) -> Resistors_SMD:R_1206_HandSoldering
- U6: footprint (none) -> footprints:SMD-8
- U7: footprint (none) -> footprints:SOT-23-5
Changed lines of the file:
@@
 EESchema Schematic File Version 2
+LIBS:stepper_driver-rescue
 LIBS:power
 LIBS:device
@@
 LIBS:custom
 LIBS:stepper_driver-cache
-EELAYER 25 0
+EELAYER 26 0
 EELAYER END
 $Descr A4 11693 8268
 encoding utf-8
 Sheet 7 10
-Title "TTL Input CMOS Output Opto Isolator"
-Date "Sun 22 Mar 2015"
+Title "Quad Stepper Motor Driver"
+Date "2016-12-15"
 Rev "1.0"
-Comp ""
+Comp "Gratian & co."
 Comment1 ""
 Comment2 ""
@@
 	4700 3800 4600 3800
 $Comp
-L GND #PWR050
+L GND #PWR053
 U 1 1 5510CB26
 P 4600 3800
-AR Path="/5510C07A/5510CB26" Ref="#PWR050"  Part="1"
-AR Path="/5515BA03/5510CB26" Ref="#PWR072"  Part="1"
-F 0 "#PWR072" H 4600 3550 50  0001 C CNN
+AR Path="/5510C07A/5510CB26" Ref="#PWR053"  Part="1"
+AR Path="/5515BA03/5510CB26" Ref="#PWR075"  Part="1"
+F 0 "#PWR075" H 4600 3550 50  0001 C CNN
 F 1 "GND" H 4600 3650 50  0000 C CNN
 F 2 "" H 4600 3800 60  0000 C CNN
@@
 F 0 "R13" V 4580 3700 50  0000 C CNN
 F 1 "390" V 4500 3700 50  0000 C CNN
-F 2 "" V 4430 3700 30  0000 C CNN
+F 2 "Resistors_SMD:R_1206_HandSoldering" V 4430 3700 30  0001 C CNN
 F 3 "" H 4500 3700 30  0000 C CNN
 	1    4500 3700
@@
 F 0 "U12" H 5150 3500 60  0000 C CNN
 F 1 "6N137S" H 5150 4000 60  0000 C CNN
-F 2 "" H 5150 3750 60  0000 C CNN
+F 2 "footprints:SMD-8" H 5150 3750 60  0001 C CNN
 F 3 "" H 5150 3750 60  0000 C CNN
 	1    5150 3750
@@
 F 0 "U13" H 6900 3500 60  0000 C CNN
 F 1 "SN74LVC1G240DBVR" H 6900 4100 60  0000 C CNN
-F 2 "" H 7000 3625 60  0000 C CNN
+F 2 "footprints:SOT-23-5" H 7000 3625 60  0001 C CNN
 F 3 "" H 7000 3625 60  0000 C CNN
 	1    6900 3800
@@
 $EndComp
 $Comp
-L GND #PWR051
+L GND #PWR054
 U 1 1 5510CB48
 P 4600 3800
-AR Path="/5510C07A/5510CB48" Ref="#PWR051"  Part="1"
-AR Path="/5515BA03/5510CB48" Ref="#PWR073"  Part="1"
-F 0 "#PWR073" H 4600 3550 50  0001 C CNN
+AR Path="/5510C07A/5510CB48" Ref="#PWR054"  Part="1"
+AR Path="/5515BA03/5510CB48" Ref="#PWR076"  Part="1"
+F 0 "#PWR076" H 4600 3550 50  0001 C CNN
 F 1 "GND" H 4600 3650 50  0000 C CNN
 F 2 "" H 4600 3800 60  0000 C CNN
@@
 	5650 3900 5750 3900
 $Comp
-L +3.3V #PWR052
+L +3.3V #PWR055
 U 1 1 55110B66
 P 5750 3450
-AR Path="/5510C07A/55110B66" Ref="#PWR052"  Part="1"
-AR Path="/5515BA03/55110B66" Ref="#PWR074"  Part="1"
-F 0 "#PWR074" H 5750 3300 50  0001 C CNN
+AR Path="/5510C07A/55110B66" Ref="#PWR055"  Part="1"
+AR Path="/5515BA03/55110B66" Ref="#PWR077"  Part="1"
+F 0 "#PWR077" H 5750 3300 50  0001 C CNN
 F 1 "+3.3V" H 5750 3590 50  0000 C CNN
 F 2 "" H 5750 3450 60  0000 C CNN
@@
 F 0 "C7" H 5175 4600 50  0000 L CNN
 F 1 "0.1uF" H 5175 4400 50  0000 L CNN
-F 2 "" H 5188 4350 30  0000 C CNN
+F 2 "Capacitors_SMD:C_1206_HandSoldering" H 5188 4350 30  0001 C CNN
 F 3 "" H 5150 4500 60  0000 C CNN
 	1    5150 4500
@@
 	5650 3800 6400 3800
 $Comp
-L GND #PWR053
+L GND #PWR056
 U 1 1 55111358
 P 6350 3950
-AR Path="/5510C07A/55111358" Ref="#PWR053"  Part="1"
-AR Path="/5515BA03/55111358" Ref="#PWR075"  Part="1"
-F 0 "#PWR075" H 6350 3700 50  0001 C CNN
+AR Path="/5510C07A/55111358" Ref="#PWR056"  Part="1"
+AR Path="/5515BA03/55111358" Ref="#PWR078"  Part="1"
+F 0 "#PWR078" H 6350 3700 50  0001 C CNN
 F 1 "GND" H 6350 3800 50  0000 C CNN
 F 2 "" H 6350 3950 60  0000 C CNN
@@
 	6350 3950 6400 3950
 $Comp
-L +3.3V #PWR054
+L +3.3V #PWR057
 U 1 1 5511153A
 P 7550 3450
-AR Path="/5510C07A/5511153A" Ref="#PWR054"  Part="1"
-AR Path="/5515BA03/5511153A" Ref="#PWR076"  Part="1"
-F 0 "#PWR076" H 7550 3300 50  0001 C CNN
+AR Path="/5510C07A/5511153A" Ref="#PWR057"  Part="1"
+AR Path="/5515BA03/5511153A" Ref="#PWR079"  Part="1"
+F 0 "#PWR079" H 7550 3300 50  0001 C CNN
 F 1 "+3.3V" H 7550 3590 50  0000 C CNN
 F 2 "" H 7550 3450 60  0000 C CNN
@@
 $EndComp
 $Comp
-L +3.3V #PWR055
+L +3.3V #PWR058
 U 1 1 5511173E
 P 5150 4300
-AR Path="/5510C07A/5511173E" Ref="#PWR055"  Part="1"
-AR Path="/5515BA03/5511173E" Ref="#PWR077"  Part="1"
-F 0 "#PWR077" H 5150 4150 50  0001 C CNN
+AR Path="/5510C07A/5511173E" Ref="#PWR058"  Part="1"
+AR Path="/5515BA03/5511173E" Ref="#PWR080"  Part="1"
+F 0 "#PWR080" H 5150 4150 50  0001 C CNN
 F 1 "+3.3V" H 5150 4440 50  0000 C CNN
 F 2 "" H 5150 4300 60  0000 C CNN
@@
 	5150 4300 5150 4350
 $Comp
-L GND #PWR056
+L GND #PWR059
 U 1 1 551117C0
 P 5150 4700
-AR Path="/5510C07A/551117C0" Ref="#PWR056"  Part="1"
-AR Path="/5515BA03/551117C0" Ref="#PWR078"  Part="1"
-F 0 "#PWR078" H 5150 4450 50  0001 C CNN
+AR Path="/5510C07A/551117C0" Ref="#PWR059"  Part="1"
+AR Path="/5515BA03/551117C0" Ref="#PWR081"  Part="1"
+F 0 "#PWR081" H 5150 4450 50  0001 C CNN
 F 1 "GND" H 5150 4550 50  0000 C CNN
 F 2 "" H 5150 4700 60  0000 C CNN
@@
 Connection ~ 5750 3600
 $Comp
-L GND #PWR057
+L GND #PWR060
 U 1 1 5510CC97
 P 5750 3900
-AR Path="/5510C07A/5510CC97" Ref="#PWR057"  Part="1"
-AR Path="/5515BA03/5510CC97" Ref="#PWR079"  Part="1"
-F 0 "#PWR079" H 5750 3650 50  0001 C CNN
+AR Path="/5510C07A/5510CC97" Ref="#PWR060"  Part="1"
+AR Path="/5515BA03/5510CC97" Ref="#PWR082"  Part="1"
+F 0 "#PWR082" H 5750 3650 50  0001 C CNN
 F 1 "GND" H 5750 3750 50  0000 C CNN
 F 2 "" H 5750 3900 60  0000 C CNN
@@
 F 0 "R14" V 6080 3650 50  0000 C CNN
 F 1 "390" V 6000 3650 50  0000 C CNN
-F 2 "" V 5930 3650 30  0000 C CNN
+F 2 "Resistors_SMD:R_1206_HandSoldering" V 5930 3650 30  0001 C CNN
 F 3 "" H 6000 3650 30  0000 C CNN
 	1    6000 3650
