File: kicad/stepper_driver/stepper_driver.sch (KiCad schematic (older format))
At the start: 11 parts, among them P1 CONN_01X10, P2 CONN_01X05, P3 CONN_01X05, P4 CONN_01X05, P5 CONN_01X05, P6 CONN_02X12, P7 CONN_01X02, U1 MCP23S18

Commit message: stepper_driver: new revision
Forgot the history on this one. If anybody is watching. Sorry :(
Moved datahseets into project folder.
I guess I've added some footprints too.

Signed-off-by: Gratian Crisan <gratian.crisan@ni.com>
Parts:
- removed P1: CONN_01X10, symbol CONN_01X10
- added D37, D38, D39: D_Schottky, Diodes_ThroughHole:Diode_DO-41_SOD81_Horizontal_RM10, symbol D_Schottky
- added P1, P10, P6, P7: 01X06, footprints:KF2EDGK-6_pin_Screw_Terminal_Block, symbol CONN_01X06
- added P11: CONN_02X03, Pin_Headers:Pin_Header_Straight_2x03, symbol CONN_02X03
- added QBX_3.3V1, QBX_GND1, SCK1, SI1, SO1, ~CS1, ~CS2, ~CS3, ~INT1, ~SO_OE1: CONN_01X01, Measurement_Points:Measurement_Point_Square-SMD-Pad_Small, symbol CONN_01X01
- added R31, R32: 150, Resistors_SMD:R_1206_HandSoldering, symbol R
- C1: footprint (none) -> Capacitors_SMD:C_1206_HandSoldering
- P2, P3, P4, P5: footprint (none) -> Terminal_Blocks:TerminalBlock_Pheonix_PT-3.5mm_5pol
- P8: renamed from P6; footprint (none) -> Connectors_Molex:Molex_MiniFit-JR-5556-24A_2x12x4.20mm_Straight; symbol CONN_02X12 -> CONN_02X12-RESCUE-stepper_driver
- P9: renamed from P7; footprint (none) -> Connect:PINHEAD1-2
- R1, R2: footprint (none) -> Resistors_SMD:R_1206_HandSoldering
- U1: footprint (none) -> SMD_Packages:SOIC-28
Connections:
- net PWR_OK is gone; now on net GND: P8.15 (P15)
- net +12V: now also P8.10 (P10), P8.11 (P11); no longer P8.19 (P19), P8.21 (P21)
- net +3V3: now also QBX_3.3V1.1 (P1); no longer P8.1 (P1), P8.2 (P2), P8.23 (P23), P8.3 (P3), R1.1
- net +5V: now also P8.4 (P4), P8.6 (P6), P9.1 (P1), R1.1, P1.6 (P6), P10.6 (P6), P6.6 (P6), P7.6 (P6); no longer P8.11 (P11), P8.18 (P18), P8.20 (P20), P8.22 (P22), P8.7 (P7)
- net -12V: no longer P8.4 (P4)
- net DRIVER0/AM0: now also P2.1 (P1); no longer P2.2 (P2)
- net DRIVER0/AM1: now also P3.1 (P1); no longer P3.2 (P2)
- net DRIVER0/AP0: now also P2.5 (P5); no longer P2.1 (P1)
- net DRIVER0/AP1: now also P3.5 (P5); no longer P3.1 (P1)
- net DRIVER0/BM0: now also P2.4 (P4); no longer P2.5 (P5)
- net DRIVER0/BM1: now also P3.4 (P4); no longer P3.5 (P5)
- net DRIVER0/BP0: now also P2.2 (P2); no longer P2.4 (P4)
- net DRIVER0/BP1: now also P3.2 (P2); no longer P3.4 (P4)
- net DRIVER1/AM0: now also P4.1 (P1); no longer P4.2 (P2)
- net DRIVER1/AM1: now also P5.1 (P1); no longer P5.2 (P2)
- net DRIVER1/AP0: now also P4.5 (P5); no longer P4.1 (P1)
- net DRIVER1/AP1: now also P5.5 (P5); no longer P5.1 (P1)
- net DRIVER1/BM0: now also P4.4 (P4); no longer P4.5 (P5)
- net DRIVER1/BM1: now also P5.4 (P4); no longer P5.5 (P5)
- net DRIVER1/BP0: now also P4.2 (P2); no longer P4.4 (P4)
- net DRIVER1/BP1: now also P5.2 (P2); no longer P5.4 (P4)
- net GND: now also P8.17 (P17), P8.18 (P18), P8.19 (P19), P8.3 (P3), P8.7 (P7), P1.5 (P5), P10.5 (P5), P11.2 (P2), P11.4 (P4), P11.6 (P6), P6.5 (P5), P7.5 (P5), QBX_GND1.1 (P1); no longer P8.10 (P10), P8.12 (P12), P8.13 (P13), P8.14 (P14), P8.6 (P6), P8.9 (P9)
- net IN_ISO_CS0/IN_CMOS: now also ~CS1.1 (P1)
- net IN_ISO_CS1/IN_CMOS: now also ~CS2.1 (P1)
- net IN_ISO_CS2/IN_CMOS: now also ~CS3.1 (P1)
- net IN_ISO_SCK/IN_CMOS: now also SCK1.1 (P1)
- net IN_ISO_SI/IN_CMOS: now also SI1.1 (P1)
- net OUT_ISO_INT/OUT_CMOS: now also ~INT1.1 (P1)
- net OUT_ISO_SO/OUT_CMOS: now also SO1.1 (P1)
- net OUT_ISO_SO/~OE: now also ~SO_OE1.1 (P1)
- net ~INT: now also D37.2 (A), D38.2 (A), D39.2 (A); no longer U1.19 (INTA)
- net at P8.16 (P16): now also P11.5 (P5)
- net at U1.10 (GPB7): now also P10.4 (P4)
- net at U1.20 (GPA0): now also P7.4 (P4)
- net at U1.21 (GPA1): now also P7.3 (P3)
- net at U1.22 (GPA2): now also P7.2 (P2)
- net at U1.23 (GPA3): now also P7.1 (P1)
- net at U1.24 (GPA4): now also P6.4 (P4)
- net at U1.25 (GPA5): now also P6.3 (P3)
- net at U1.26 (GPA6): now also P6.2 (P2)
- net at U1.27 (GPA7): now also P6.1 (P1)
- net at U1.3 (GPB0): now also P1.1 (P1)
- net at U1.4 (GPB1): now also P1.2 (P2)
- net at U1.5 (GPB2): now also P1.3 (P3)
- net at U1.6 (GPB3): now also P1.4 (P4)
- net at U1.7 (GPB4): now also P10.1 (P1)
- net at U1.8 (GPB5): now also P10.2 (P2)
- net at U1.9 (GPB6): now also P10.3 (P3)
- removed net 5V_STBY: P8.17 (P17), P9.1 (P1)
- net NC: no longer names the net of U1.18 (INTB)
- net ~PSon: no longer names the net of P8.8 (P8)
- net ~PSon: now also R32.2
- new net: P8.9 (P9), R31.2
- new net: D39.1 (K), U1.19 (INTA)
- new net: P11.3 (P3), R31.1
- new net: P11.1 (P1), R32.1
- new net DRIVER0/INT: D37.1 (K)
- new net DRIVER1/INT: D38.1 (K)
- no-connect marks 0 -> 10
